File: placa IOT/Alimentacion.kicad_sch (KiCad schematic)
At the start: 0 parts

Commit message: ALIMENTACION
Parts:
- added C1, C2, C3, C4: 100nF, Capacitor_SMD:C_0402_1005Metric, symbol Device:C
- added R2, R3: 10K, Resistor_SMD:R_0402_1005Metric, symbol Device:R
- added R4: NC R22, Resistor_SMD:R_0402_1005Metric, symbol Device:R
- added U1, U2: RT9080-33GJ5, ic_power:TSOT-23-5_RIT, symbol ic_power:RT9080-33GJ5
Connections:
- new net: R2.2, U1.3 (EN)
- new net: R3.2, R4.2, U2.3 (EN)
- new net +3.3V: C2.1, C3.1, U1.5 (VOUT), U2.5 (VOUT)
- new net +5V: C1.1, C4.1, R2.1, R3.1, U1.1 (VIN), U2.1 (VIN)
- new net GND: C1.2, C2.2, C3.2, C4.2, U1.2 (GND), U2.2 (GND)
