File: placa IOT/placa IOT.kicad_sch (KiCad schematic)
At the start: 0 parts

Commit message: ESQUEMATICO AÑADIDO
Other:
- added sheet Alimentacion (Alimentacion.kicad_sch)
- added sheet Bateria (Bateria.kicad_sch)
- added sheet MCU_WIFIBLU (MCU_WIFIBLU.kicad_sch)
- added sheet RF_LORA (RF_LORA.kicad_sch)
- company: (none) -> ELE0226CL
- title: (none) -> BLOQUE ALIMENTACIÓN
Changed lines of the file:
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@@
 	(generator "eeschema")
 	(generator_version "10.0")
-	(paper "A4")
+	(paper "A3")
+	(title_block
+		(title "BLOQUE ALIMENTACIÓN")
+		(date "19/05/2026")
+		(rev "Mª Angeles Lolo")
+		(company "ELE0226CL")
+	)
+	(sheet
+		(at 257.81 40.64)
+		(size 135.89 100.33)
+		(exclude_from_sim no)
+		(in_bom yes)
+		(on_board yes)
+		(dnp no)
+		(fields_autoplaced yes)
+		(stroke
+			(width 0.1524)
+			(type solid)
+		)
+		(fill
+			(color 0 0 0 0)
+		)
+		(property "Sheetname" "Bateria"
+			(at 257.81 39.9284 0)
+			(show_name no)
+			(do_not_autoplace no)
+			(effects
+				(font
+					(size 1.27 1.27)
+				)
+				(justify left bottom)
+			)
+		)
+		(property "Sheetfile" "Bateria.kicad_sch"
+			(at 257.81 141.5546 0)
+			(show_name no)
+			(do_not_autoplace no)
+			(effects
+				(font
+					(size 1.27 1.27)
+				)
+				(justify left top)
+			)
+		)
+		(instances
+			(project "placa IOT"
+				(path "/fbbb61cd-c6c4-4d51-9fb8-e36c0f4e7910"
+					(page "5")
+				)
+			)
+		)
+	)
+	(sheet
+		(at 44.45 132.08)
+		(size 73.66 88.9)
+		(exclude_from_sim no)
+		(in_bom yes)
+		(on_board yes)
+		(dnp no)
+		(fields_autoplaced yes)
+		(stroke
+			(width 0.1524)
+			(type solid)
+		)
+		(fill
+			(color 0 0 0 0)
+		)
+		(property "Sheetname" "RF_LORA"
+			(at 44.45 131.3684 0)
+			(show_name no)
+			(do_not_autoplace no)
+			(effects
+				(font
+					(size 1.27 1.27)
+				)
+				(justify left bottom)
+			)
+		)
+		(property "Sheetfile" "RF_LORA.kicad_sch"
+			(at 44.45 221.5646 0)
+			(show_name no)
+			(do_not_autoplace no)
+			(effects
+				(font
+					(size 1.27 1.27)
+				)
+				(justify left top)
+			)
+		)
+		(instances
+			(project "placa IOT"
+				(path "/fbbb61cd-c6c4-4d51-9fb8-e36c0f4e7910"
+					(page "4")
+				)
+			)
+		)
+	)
+	(sheet
+		(at 68.58 40.64)
+		(size 45.72 43.18)
+		(exclude_from_sim no)
+		(in_bom yes)
+		(on_board yes)
+		(dnp no)
+		(fields_autoplaced yes)
+		(stroke
+			(width 0.1524)
+			(type solid)
+		)
+		(fill
+			(color 0 0 0 0)
+		)
+		(property "Sheetname" "Alimentacion"
+			(at 68.58 39.9284 0)
+			(show_name yes)
+			(do_not_autoplace no)
+			(effects
+				(font
+					(size 1.27 1.27)
+				)
+				(justify left bottom)
+			)
+		)
+		(property "Sheetfile" "Alimentacion.kicad_sch"
+			(at 68.58 84.4046 0)
+			(show_name no)
+			(do_not_autoplace no)
+			(effects
+				(font
+					(size 1.27 1.27)
+				)
+				(justify left top)
+			)
+		)
+		(instances
+			(project "placa IOT"
+				(path "/fbbb61cd-c6c4-4d51-9fb8-e36c0f4e7910"
+					(page "2")
+				)
+			)
+		)
+	)
+	(sheet
+		(at 180.34 40.64)
+		(size 41.91 162.56)
+		(exclude_from_sim no)
+		(in_bom yes)
+		(on_board yes)
+		(dnp no)
+		(fields_autoplaced yes)
+		(stroke
+			(width 0.1524)
+			(type solid)
+		)
+		(fill
+			(color 0 0 0 0)
+		)
+		(property "Sheetname" "MCU_WIFIBLU"
+			(at 180.34 39.9284 0)
+			(show_name no)
+			(do_not_autoplace no)
+			(effects
+				(font
+					(size 1.27 1.27)
+				)
+				(justify left bottom)
+			)
+		)
+		(property "Sheetfile" "MCU_WIFIBLU.kicad_sch"
+			(at 180.34 203.7846 0)
+			(show_name no)
+			(do_not_autoplace no)
+			(effects
+				(font
+					(size 1.27 1.27)
+				)
+				(justify left top)
+			)
+		)
+		(instances
+			(project "placa IOT"
+				(path "/fbbb61cd-c6c4-4d51-9fb8-e36c0f4e7910"
+					(page "3")
+				)
+			)
+		)
+	)
 	(sheet_instances
 		(path "/"

Commit message: USB TERMINADO
Other:
- added sheet USB (USB.kicad_sch)
Changed lines of the file:
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@@
+		)
+	)
+	(sheet
+		(at 259.08 161.29)
+		(size 133.35 64.77)
+		(exclude_from_sim no)
+		(in_bom yes)
+		(on_board yes)
+		(dnp no)
+		(fields_autoplaced yes)
+		(stroke
+			(width 0.1524)
+			(type solid)
+		)
+		(fill
+			(color 0 0 0 0)
+		)
+		(property "Sheetname" "USB"
+			(at 259.08 160.5784 0)
+			(show_name no)
+			(do_not_autoplace no)
+			(effects
+				(font
+					(size 1.27 1.27)
+				)
+				(justify left bottom)
+			)
+		)
+		(property "Sheetfile" "USB.kicad_sch"
+			(at 259.08 226.6446 0)
+			(show_name no)
+			(do_not_autoplace no)
+			(effects
+				(font
+					(size 1.27 1.27)
+				)
+				(justify left top)
+			)
+		)
+		(instances
+			(project "placa IOT"
+				(path "/fbbb61cd-c6c4-4d51-9fb8-e36c0f4e7910"
+					(page "6")
+				)
+			)
 		)
 	)

Commit message: ACABADO
Other:
- sheet Bateria ports: added ID1, IO4, VBAT; removed none
- sheet MCU_WIFIBLU ports: added D+, D-, ID1, IO3, IO33, IO34, IO36, IO4, IO5, IO6, IO7, IO8, IO9, LORA_RX, LORA_TX; removed none
- sheet RF_LORA ports: added 3.3VP, IO3, IO33, IO34, IO36, IO5, IO6, IO7, IO8, IO9, LORA_RX, LORA_TX; removed none
- sheet USB ports: added D+, D-; removed none
