File: placa IOT/Bateria.kicad_sch (KiCad schematic)
At the start: 0 parts

Commit message: MICROCONTROLADOR TERMINADOCON CAMBIO
Parts:
- added D1: SS34, Diode_SMD:D_SMA, symbol Diode:SS34
- added Q1: PMOS, symbol Simulation_SPICE:PMOS
- added R10: 499 OHM, Resistor_SMD:R_0402_1005Metric, symbol Device:R
Connections:
- new net: D1.1 (K), Q1.3 (S)
- new net VBAT: Q1.1 (D)
- new net VBUS: D1.2 (A), Q1.2 (G), R10.1

Commit message: USB TERMINADO
Parts:
- added C25, C27: 10uF, Capacitor_SMD:C_0402_1005Metric, symbol Device:C
- added C26, C28: 100nF, Capacitor_SMD:C_0402_1005Metric, symbol Device:C
- added D2: D_Zener, Diode_SMD:D_SOD-123, symbol Device:D_Zener
- added D3: LED BLUE, LED_SMD:LED_0402_1005Metric, symbol Device:LED
- added D4: LED RED, LED_SMD:LED_0402_1005Metric, symbol Device:LED
- added D5: SS34, Diode_SMD:D_SMA, symbol Diode:SS34
- added J4: 620102131822, connectors:CONN_SMT_MH_SH_P2.00MM_P2, symbol connectors:CONN_SMT_MH_SH_P2.00MM_P2
- added J5: B2B-PH-K-S(LF)(SN), connectors:CONN_THT_MV_JST_P2.00MM_P2, symbol connectors:CONN_THT_MV_JST_P2.00MM_P2
- added Q2: PMOS, symbol Simulation_SPICE:PMOS
- added R14, R15, R20, R21: 100K, Resistor_SMD:R_0402_1005Metric, symbol Device:R
- added R16, R17: 1K, Resistor_SMD:R_0402_1005Metric, symbol Device:R
- added R18: 2K, Resistor_SMD:R_0402_1005Metric, symbol Device:R
- added R19: 0, Resistor_SMD:R_0402_1005Metric, symbol Device:R
- added R22: 10K, Resistor_SMD:R_0402_1005Metric, symbol Device:R
- added SW3, SW4: SW_DPDT_x2, symbol Switch:SW_DPDT_x2
- added U6: CN3065, ic_power:DFN-8-1EP_3x3mm_P0.5mm_EP1.66x2.38mm, symbol ic_power:CN3065
- R10: value 499 OHM -> 10K
Connections:
- net VBAT: now also C27.1, J4.1 (Pin_1), Q2.1 (D), R20.1, U6.5 (BAT), U6.8 (FB)
- net at D1.1 (K), Q1.3 (S): now also SW3.2 (B)
- net GND: now reaches R10.2
- net GND: now also C25.2, C26.2, C27.2, C28.2, D2.2 (A), J4.2 (Pin_2), J5.1 (Pin_1), R15.2, R18.2, R19.2, R21.2, R22.2, U6.3 (GND), U6.9 (GND)
- net VBUS renamed SOLAR
- net SOLAR: now also D2.1 (K), D5.2 (A), J5.2 (Pin_2), Q2.2 (G), R14.1, R22.1
- new net: D5.1 (K), Q2.3 (S), SW4.2 (B)
- new net: R19.1, U6.1 (TEMP)
- new net: R18.1, U6.2 (ISET)
- new net: C25.1, C26.1, R16.1, R17.1, U6.4 (VIN)
- new net: D3.1 (K), U6.6 (~{DONE})
- new net: D4.1 (K), U6.7 (~{CHRG})
- new net: D3.2 (A), R16.2
- new net: D4.2 (A), R17.2
- new net 5V: SW3.1 (A), SW4.1 (A)
- new net ID1: C28.1, R20.2, R21.1
- new net IO4: R14.2, R15.1
- no-connect marks 0 -> 2
Other:
- moved on the sheet: D1, Q1, R10

Commit message: ACABADO
Connections:
- net VBAT: no longer C27.1, J4.1 (Pin_1), R20.1, U6.5 (BAT), U6.8 (FB)
- new net: C27.1, J4.1 (Pin_1), R20.1, U6.5 (BAT), U6.8 (FB)
Changed lines of the file:
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@@
-	)
-	(junction
-		(at 262.89 82.55)
-		(diameter 0)
-		(color 0 0 0 0)
 	)
 	(junction
@@
 	(wire
 		(pts
-			(xy 250.19 104.14) (xy 271.78 104.14)
+			(xy 250.19 82.55) (xy 262.89 82.55)
 		)
 		(stroke
@@
 	(wire
 		(pts
-			(xy 250.19 82.55) (xy 262.89 82.55)
-		)
-		(stroke
-			(width 0)
-			(type default)
-		)
-	)
-	(wire
-		(pts
 			(xy 260.35 115.57) (xy 271.78 115.57)
 		)
@@
 	(wire
 		(pts
-			(xy 262.89 82.55) (xy 264.16 82.55)
-		)
-		(stroke
-			(width 0)
-			(type default)
-		)
-	)
-	(wire
-		(pts
 			(xy 226.06 127) (xy 226.06 130.81)
 		)
@@
 	(wire
 		(pts
-			(xy 80.01 144.78) (xy 110.49 144.78)
-		)
-		(stroke
-			(width 0)
-			(type default)
-		)
-	)
-	(wire
-		(pts
 			(xy 219.71 101.6) (xy 232.41 101.6)
 		)
@@
 	)
 	(hierarchical_label "ID1"
-		(shape input)
+		(shape output)
 		(at 271.78 115.57 0)
 		(effects
@@
 	)
 	(hierarchical_label "IO4"
-		(shape input)
+		(shape output)
 		(at 49.53 52.07 180)
 		(effects
@@
 		)
 	)
-	(hierarchical_label "VBAT"
-		(shape input)
-		(at 271.78 104.14 0)
-		(effects
-			(font
-				(size 1.27 1.27)
-			)
-			(justify left)
-		)
-	)

Commit message: ULTIMA  PRUEBA
Parts:
- Q1, Q2: footprint (none) -> Package_TO_SOT_SMD:SOT-23-3
- SW4: footprint (none) -> Button_Switch_THT:SW_Slide_SPDT_Angled_CK_OS102011MA1Q
Changed lines of the file:
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@@
 			)
 		)
-		(property "Footprint" ""
+		(property "Footprint" "Button_Switch_THT:SW_Slide_SPDT_Angled_CK_OS102011MA1Q"
 			(at 78.74 160.02 0)
 			(hide yes)
@@
 			)
 		)
-		(property "Footprint" ""
+		(property "Footprint" "Package_TO_SOT_SMD:SOT-23-3"
 			(at 110.49 59.69 0)
 			(hide yes)
@@
 			)
 		)
-		(property "Footprint" ""
+		(property "Footprint" "Package_TO_SOT_SMD:SOT-23-3"
 			(at 81.28 125.73 0)
 			(hide yes)

Commit message: ULTIMA PRUEBA2
Parts:
- removed SW3: SW_DPDT_x2, symbol Switch:SW_DPDT_x2
- added SW5: SW_DPDT_x2, Button_Switch_THT:SW_Slide_SPDT_Angled_CK_OS102011MA1Q, symbol Switch:SW_DPDT_x2
Connections:
- net 5V: now also SW5.1 (A)
- net at D1.1 (K), Q1.3 (S): now also SW5.2 (B)
Changed lines of the file:
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@@
+	)
+	(symbol
+		(lib_id "Switch:SW_DPDT_x2")
+		(at 107.95 93.98 270)
+		(unit 1)
+		(body_style 1)
+		(exclude_from_sim no)
+		(in_bom yes)
+		(on_board yes)
+		(in_pos_files yes)
+		(dnp no)
+		(fields_autoplaced yes)
+		(property "Reference" "SW5"
+			(at 113.03 92.7099 90)
+			(show_name no)
+			(do_not_autoplace no)
+			(effects
+				(font
+					(size 1.27 1.27)
+				)
+				(justify left)
+			)
+		)
+		(property "Value" "SW_DPDT_x2"
+			(at 113.03 95.2499 90)
+			(show_name no)
+			(do_not_autoplace no)
+			(effects
+				(font
+					(size 1.27 1.27)
+				)
+				(justify left)
+			)
+		)
+		(property "Footprint" "Button_Switch_THT:SW_Slide_SPDT_Angled_CK_OS102011MA1Q"
+			(at 107.95 93.98 0)
+			(hide yes)
+			(show_name no)
+			(do_not_autoplace no)
+			(effects
+				(font
+					(size 1.27 1.27)
+				)
+			)
+		)
+		(property "Datasheet" ""
+			(at 107.95 93.98 0)
+			(hide yes)
+			(show_name no)
+			(do_not_autoplace no)
+			(effects
+				(font
+					(size 1.27 1.27)
+				)
+			)
+		)
+		(property "Description" "Switch, dual pole double throw, separate symbols"
+			(at 107.95 93.98 0)
+			(hide yes)
+			(show_name no)
+			(do_not_autoplace no)
+			(effects
+				(font
+					(size 1.27 1.27)
+				)
+			)
+		)
+		(pin "6"
+		)
+		(pin "5"
+		)
+		(pin "2"
+		)
+		(pin "3"
+		)
+		(pin "4"
+		)
+		(pin "1"
+		)
+		(instances
+			(project "placa IOT"
+				(path "/fbbb61cd-c6c4-4d51-9fb8-e36c0f4e7910/04ee4292-769c-446c-ae88-043e80bec59b"
+					(reference "SW5")
+					(unit 1)
+				)
+			)
+		)
 	)
 	(symbol
@@
 					(unit 1)
 				)
-			)
-		)
-	)
-	(symbol
-		(lib_id "Switch:SW_DPDT_x2")
-		(at 107.95 93.98 270)
-		(unit 1)
-		(body_style 1)
-		(exclude_from_sim no)
-		(in_bom yes)
-		(on_board yes)
-		(in_pos_files yes)
-		(dnp no)
-		(fields_autoplaced yes)
-		(property "Reference" "SW3"
-			(at 113.03 92.7099 90)
-			(show_name no)
-			(do_not_autoplace no)
-			(effects
-				(font
-					(size 1.27 1.27)
-				)
-				(justify left)
-			)
-		)
-		(property "Value" "SW_DPDT_x2"
-			(at 113.03 95.2499 90)
-			(show_name no)
-			(do_not_autoplace no)
-			(effects
-				(font
-					(size 1.27 1.27)
-				)
-				(justify left)
-			)
-		)
-		(property "Footprint" ""
-			(at 107.95 93.98 0)
-			(hide yes)
-			(show_name no)
-			(do_not_autoplace no)
-			(effects
-				(font
-					(size 1.27 1.27)
-				)
-			)
-		)
-		(property "Datasheet" ""
-			(at 107.95 93.98 0)
-			(hide yes)
-			(show_name no)
-			(do_not_autoplace no)
-			(effects
-				(font
-					(size 1.27 1.27)
-				)
-			)
-		)
-		(property "Description" "Switch, dual pole double throw, separate symbols"
-			(at 107.95 93.98 0)
-			(hide yes)
-			(show_name no)
-			(do_not_autoplace no)
-			(effects
-				(font
-					(size 1.27 1.27)
-				)
-			)
-		)
-		(pin "6"
-		)
-		(pin "5"
-		)
-		(pin "2"
-		)
-		(pin "3"
-		)
-		(pin "4"
-		)
-		(pin "1"
-		)
-		(instances
-			(project "placa IOT"
-				(path "/fbbb61cd-c6c4-4d51-9fb8-e36c0f4e7910/04ee4292-769c-446c-ae88-043e80bec59b"
-					(reference "SW3")
-					(unit 1)
-				)
