File: placa IOT/placa IOT.kicad_pcb (KiCad board)
At the start: 4 copper layers, 85 parts, among them J1 22-28-4144, J2 22-28-4144, J3 20279-001E-03, J4 620102131822, J5 B2B-PH-K-S(LF)(SN), J6 USB4105-GF-A-120, Q1 PMOS, Q2 PMOS, SW1 RST/EN, SW2 BOOT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

Commit message: ULTIMA PRUEBA2
Parts:
- added M1: MountingHole_2.5mm_Pad_TopBottom, MountingHole:MountingHole_2.5mm_Pad_TopBottom, F.Cu at (16.7, 40.6)
- added M2: MountingHole_2.5mm_Pad_TopBottom, MountingHole:MountingHole_2.5mm_Pad_TopBottom, F.Cu at (65.7, 40.3)
- added M3: MountingHole_2.5mm_Pad_TopBottom, MountingHole:MountingHole_2.5mm_Pad_TopBottom, F.Cu at (16.8, 164.2)
- added M4: MountingHole_2.5mm_Pad_TopBottom, MountingHole:MountingHole_2.5mm_Pad_TopBottom, F.Cu at (65.7, 164.1)
- moved C1 193.0 mm to (27.9, 52.8), turned to 90 degrees
- moved C2 191.3 mm to (30.8, 52.8), turned to 90 degrees
- moved C3 190.4 mm to (32.8, 52.8), turned to 90 degrees
- moved C4 189.5 mm to (34.7, 52.8), turned to 90 degrees
- moved R7 186.3 mm to (29.6, 99.2), turned to 90 degrees
- moved J3 183.5 mm to (15.9, 131.9)
- moved U5 180.3 mm to (32.9, 89.2), turned to 180 degrees
- moved R11 178.9 mm to (36.8, 84.1), turned to 90 degrees
- moved R2 176.9 mm to (29.3, 115.8)
- moved R12 175.9 mm to (39.9, 84.1), turned to 90 degrees
- moved R13 173.1 mm to (42.8, 84.1), turned to 90 degrees
- moved C26 172.6 mm to (43.8, 140.4)
- moved C25 172.5 mm to (43.9, 138.4)
- moved R3 172.1 mm to (34.4, 115.8)
- moved D3 171.3 mm to (44.6, 143.6)
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Other:
- board outline added: 57 x 132 mm
